File: Regulator.kicad_pcb (KiCad board)
At the start: 2 copper layers, 26 parts, among them J1 Conn_01x04_Pin, Q1 D965L, Q2 C1815L, Q3 C1815L, Q4 TIP107, Q5 A1015L

Commit message: Routing and layout done
Parts:
- added J2: Conn_01x01_Pin, Connector_Wire:SolderWire-6sqmm_1x01_D3.5mm_OD7mm, F.Cu at (145.9, 117.0)
- added J3: Conn_01x01_Pin, Connector_Wire:SolderWire-6sqmm_1x01_D3.5mm_OD7mm, F.Cu at (154.9, 117.0)
- added J4: Conn_01x01_Pin, Connector_Wire:SolderWire-6sqmm_1x01_D3.5mm_OD7mm, F.Cu at (164.0, 117.0)
- added J5: Conn_01x01_Pin, Connector_Wire:SolderWire-6sqmm_1x01_D3.5mm_OD7mm, F.Cu at (179.0, 117.0)
- J1: value Conn_01x04_Pin -> Conn_01x01_Pin; footprint Connector_PinHeader_2.54mm:PinHeader_1x04_P2.54mm_Vertical -> Connector_Wire:SolderWire-6sqmm_1x01_D3.5mm_OD7mm
- R1, R10, R12, R13, R14, R3, R4, R5, R6, R8: footprint Resistor_THT:R_Axial_DIN0204_L3.6mm_D1.6mm_P5.08mm_Horizontal -> Resistor_THT:R_Axial_DIN0207_L6.3mm_D2.5mm_P10.16mm_Horizontal
- R11, R2, R7: footprint Resistor_THT:R_Axial_DIN0204_L3.6mm_D1.6mm_P5.08mm_Horizontal -> Resistor_THT:R_Axial_DIN0309_L9.0mm_D3.2mm_P15.24mm_Horizontal
- R9: value 100 ? -> 10; footprint Resistor_THT:R_Axial_DIN0204_L3.6mm_D1.6mm_P5.08mm_Horizontal -> Resistor_THT:R_Axial_DIN0516_L15.5mm_D5.0mm_P20.32mm_Horizontal
- moved Q1 104.8 mm to (181.2, 71.9)
- moved Q2 104.0 mm to (181.2, 80.9)
- moved R11 87.3 mm to (176.5, 109.6), turned to 90 degrees
- moved R9 83.1 mm to (182.5, 109.2), turned to 90 degrees
- moved Q3 79.2 mm to (152.7, 78.4)
- moved R10 78.9 mm to (168.5, 99.4), turned to -90 degrees
- moved R5 78.2 mm to (174.0, 80.6), turned to 90 degrees
- moved R4 73.9 mm to (170.5, 80.6), turned to 90 degrees
- moved R8 72.9 mm to (172.5, 109.6), turned to 90 degrees
- moved R6 72.7 mm to (167.0, 80.6), turned to 90 degrees
- moved R13 69.1 mm to (155.0, 85.0)
- moved R12 66.9 mm to (154.9, 89.5)
- moved R3 66.3 mm to (163.5, 80.6), turned to 90 degrees
- moved Q5 65.3 mm to (143.7, 102.5)
- moved C2 64.9 mm to (153.0, 69.5)
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Connections:
- C1 pad 1: Net-(Q4-B) -> Net-(D3-K)
- C1 pad 2: Net-(D3-K) -> Net-(Q4-B)
Routing:
- net A: track 0.00 -> 73.0 mm
- net Net-(Q4-B): track 0.00 -> 65.0 mm
- net Net-(Q1-B): track 0.00 -> 57.0 mm
- net Net-(Q2-B): track 0.00 -> 51.7 mm
- net Net-(D3-A): track 0.00 -> 43.9 mm
- net I: track 0.00 -> 41.3 mm
- net F: track 0.00 -> 36.4 mm
- net Net-(D2-K): track 0.00 -> 28.8 mm
- net Net-(Q2-C): track 0.00 -> 26.1 mm
- net Net-(D3-K): track 0.00 -> 23.8 mm
- net Net-(Q1-C): track 0.00 -> 19.0 mm
- net Net-(Q3-B): track 0.00 -> 16.1 mm
- net GND: track 0.00 -> 13.1 mm
- net Net-(D2-A): track 0.00 -> 6.12 mm
- net Net-(C3-Pad1): track 0.00 -> 5.00 mm
- added copper zone on B.Cu, net GND
- added copper zone on F.Cu, net GND
Other:
- board outline added: 65 x 62 mm

Commit message: Started simulation work for circuit
Parts:
- removed D1, D2: 1N4007, Diode_THT:D_A-405_P7.62mm_Horizontal
- removed Q2, Q3: C1815L, Package_TO_SOT_THT:TO-92_Inline
- removed Q4: TIP107, Package_TO_SOT_THT:TO-220-3_Vertical
- removed Q5: A1015L, Package_TO_SOT_THT:TO-92_Inline
- added D4: 1N4007, Diode_THT:D_DO-41_SOD81_P10.16mm_Horizontal, F.Cu at (144.5, 69.5)
- added D5: 1N4007, Diode_THT:D_DO-41_SOD81_P10.16mm_Horizontal, F.Cu at (135.5, 80.1)
- added Q6: BC547, Package_TO_SOT_THT:TO-92_Inline, F.Cu at (174.5, 75.5)
- added Q7: BC557, Package_TO_SOT_THT:TO-92_Inline, F.Cu at (145.5, 103.5)
- added Q8: BD139, Package_TO_SOT_THT:TO-126-3_Vertical, F.Cu at (181.5, 75.5)
- added Q9: TIP127, Package_TO_SOT_THT:TO-220-3_Vertical, F.Cu at (134.4, 109.0)
- D3: value D_Zener -> 6.5V
- Q1: value D965L -> BC547
- moved Q1 33.0 mm to (149.0, 79.0)
- moved R5 16.3 mm to (162.5, 69.0), turned to -90 degrees
- moved R3 4.74 mm to (159.0, 79.1)
- moved R9 4.30 mm to (184.0, 105.2)
- moved R10 4.30 mm to (170.0, 95.4)
- moved R11 4.30 mm to (178.0, 105.6)
- moved R8 4.30 mm to (174.0, 105.6)
- moved D3 2.08 mm to (157.5, 99.7)
- moved R4 1.80 mm to (169.5, 79.1)
- moved R6 1.80 mm to (166.0, 79.1)
- moved R14 1.44 mm to (153.5, 108.6)
- moved C2 1.11 mm to (152.0, 69.0), turned to -90 degrees
Connections:
- net Net-(D3-A) renamed /anode
- net Net-(D3-K) renamed /cathode
- J2 pad 1: S -> A
- Q1 pad 1: GND -> Net-(Q1-C)
- Q1 pad 2: Net-(Q1-C) -> Net-(Q1-B)
- Q1 pad 3: Net-(Q1-B) -> GND
- R10 pad 1: Net-(Q2-C) -> Net-(Q1-C)
- R11 pad 2: Net-(Q2-C) -> Net-(Q1-C)
- R2 pad 1: Net-(D2-A) -> A
- R3 pad 1: Net-(Q2-B) -> Net-(Q1-B)
- R5 pad 2: Net-(Q2-B) -> Net-(Q1-B)
- R7 pad 2: Net-(Q1-B) -> Net-(Q6-C)
- R8 pad 2: Net-(Q2-B) -> Net-(Q1-B)
- R9 pad 2: Net-(Q1-C) -> Net-(Q8-C)
Routing:
- net A: track 73.0 -> 0.00 mm
- net Net-(Q7-C): track 65.0 -> 0.00 mm
- net Net-(Q1-B): track 57.0 -> 0.00 mm
- net Net-(Q2-B): track 51.7 -> 0.00 mm
- net /anode: track 43.9 -> 0.00 mm
- net I: track 41.3 -> 0.00 mm
- net F: track 36.4 -> 0.00 mm
- net Net-(D4-K): track 28.8 -> 0.00 mm
- net Net-(Q2-C): track 26.1 -> 0.00 mm
- net /cathode: track 23.8 -> 0.00 mm
- net Net-(Q1-C): track 19.0 -> 0.00 mm
- net Net-(Q6-B): track 16.1 -> 0.00 mm
- net GND: track 13.1 -> 0.00 mm
- net Net-(D2-A): track 6.12 -> 0.00 mm
- net Net-(C3-Pad1): track 5.00 -> 0.00 mm

Commit message: Production ready prototype
Parts:
- D3: value 6.5V -> Vz = 6.5V
- moved Q8 6.06 mm to (186.3, 79.2), turned to 180 degrees
- moved D5 3.95 mm to (131.6, 80.0)
- moved R14 3.06 mm to (153.4, 105.5)
- moved D3 2.98 mm to (159.4, 97.4)
- moved Q9 2.45 mm to (132.5, 107.5)
- moved J1 2.00 mm to (136.8, 119.0)
- moved J2 2.00 mm to (145.9, 119.0)
- moved J3 2.00 mm to (154.9, 119.0)
- moved J4 2.00 mm to (164.0, 119.0)
- moved J5 2.00 mm to (179.0, 119.0)
- moved R7 1.81 mm to (164.0, 108.6)
- moved C1 1.79 mm to (149.0, 92.2)
- moved Q1 1.58 mm to (150.6, 79.0)
- moved R2 1.06 mm to (138.9, 82.3)
- moved D4 0.64 mm to (145.1, 69.7)
Connections:
- D4 pad 2: A -> S
- J2 pad 1: A -> S
- R2 pad 1: A -> S
Routing:
- net A: track 0.00 -> 81.2 mm
- net Net-(Q7-C): track 0.00 -> 61.5 mm
- net F: track 0.00 -> 55.8 mm
- net S: track 0.00 -> 46.8 mm
- net I: track 0.00 -> 39.3 mm
- net /anode: track 0.00 -> 39.1 mm
- net Net-(Q1-C): track 0.00 -> 38.7 mm
- net Net-(Q1-B): track 0.00 -> 33.4 mm
- net Net-(Q6-C): track 0.00 -> 31.0 mm
- net Net-(D4-K): track 0.00 -> 26.0 mm
- net /cathode: track 0.00 -> 23.4 mm
- net Net-(Q6-B): track 0.00 -> 12.3 mm
- net Net-(Q8-C): track 0.00 -> 5.62 mm
- net Net-(C3-Pad1): track 0.00 -> 5.00 mm
Other:
- board text added: "F S A I GND"
- board text added: "REVR Rev-A PROTOYPE, NOT FOR RESALE NO REGULATORY APPROVAL USE AT OWN RISK EVALUATION ONLY DESIGNED BY INDOOR_INDUSTRY 05/2026"
